File: Baja_ECVT_controller.kicad_sch (KiCad schematic)
At the start: 37 parts, among them J1 Conn_01x04_Pin, J3 USB_C_Receptacle_USB2.0, J4 Micro_SD_Card_Det2, SW1 SW_Push, SW2 SW_SPDT, U1 STM32H725VGT6, U7 SN65HVD230, Y1 TSX-3225_16.0000MF09Z-AC6

Commit message: Add files via upload
Parts:
- added C41, C42: 100n, symbol Device:C
- added R7: 10k, symbol Device:R
- added U9: SN74LVC1T45DBV, Package_TO_SOT_SMD:SOT-23-6, symbol Logic_LevelTranslator:SN74LVC1T45DBV
Connections:
- net +3.3V: now also C42.2, U9.6 (VCCB)
- net GND: now also C41.2, C42.1, U9.2 (GND)
- net Encoder1_1: no longer names the net of U1.67 (PA9)
- net Encoder1_2 renamed Hall_effect_3.3v
- net Hall_effect_3.3v: now also U9.4 (B)
- new net: R7.1, U9.5 (DIR)
- new net +5V: C41.1, R7.2, U9.1 (VCCA)
- new net Hall_Effect: U9.3 (A)
Other:
- note added: "Hall Effect Level Shifting"

Commit message: Add files via upload
Parts:
- added H1, H2, H3, H4: MountingHole, MountingHole:MountingHole_3.2mm_M3, symbol Mechanical:MountingHole
- C1, C10, C11, C12, C15, C16, C17, C19, C2, C3, C38, C4, C41, C42, C5, C6, C7, C8: footprint (none) -> Capacitor_SMD:C_0402_1005Metric
- C13, C20: footprint (none) -> Capacitor_SMD:C_0805_2012Metric
- C14, C18, C21, C22, C23: footprint (none) -> Capacitor_SMD:C_0603_1608Metric
- J1: footprint (none) -> Connector_PinHeader_2.54mm:PinHeader_1x04_P2.54mm_Vertical
- J3: footprint (none) -> Connector_USB:USB_C_Receptacle_Amphenol_12401610E4-2A
- J4: footprint (none) -> Connector_Card:microSD_HC_Hirose_DM3D-SF
- L1: footprint (none) -> Inductor_SMD:L_0603_1608Metric
- R1, R2, R27, R3, R4, R7: footprint (none) -> Resistor_SMD:R_0402_1005Metric
- SW1: footprint (none) -> Button_Switch_SMD:SW_Tactile_SPST_NO_Straight_CK_PTS636Sx25SMTRLFS
- SW2: footprint (none) -> Button_Switch_SMD:SW_SPDT_CK-JS102011SAQN
- U1: footprint LQFP100_14X14_STM -> Package_QFP:LQFP-100_14x14mm_P0.5mm
- Y1: footprint TSX-3225_16.0000MF09Z-AC6:XTAL_TSX-3225_16.0000MF09Z-AC6 -> Crystal:XTAL_TSX-3225_16.0000MF09Z-AC6
Connections:
- net Current_sense_2: no longer names the net of U1.35 (PC4)
- net Encoder3_1 renamed Encoder1_1
- net Encoder3_2 renamed Encoder1_2
