File: batt_indc.kicad_sch (KiCad schematic)
At the start: 17 parts, among them Q1 PMOS, Q2 PMOS, U3 LM393

Commit message: Add files via upload
Parts:
- removed R10, R13: 4k7, symbol Device:R
- removed R14: 6k8, symbol Device:R
- removed R9: 2k2, symbol Device:R
- added RV1, RV2: 10k, symbol Device:R_Potentiometer
- R11, R15: value 8k2 -> 100k
- R12, R16: value 2k2 -> 10k
- R17, R18: value 2k2 -> 220
Connections:
- net +5V: now also RV1.1, RV2.1
- net GND: now also RV1.3, RV2.3
- net at U3.6 (-): now also RV1.2
- net at U3.2 (-): now also RV2.2
Other:
- note added: "Dead Battery warning, adjustable"
- note added: "Low Battery Warning, adjustable"
- note removed: "Dead Battery warning triggers at 2.79v/cell"
- note removed: "Low voltage warning triggers at 3.22v/cell"
Changed lines of the file:
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@@
 (kicad_sch (version 20230121) (generator eeschema)
   (paper "A4")
-  (junction (at 109.22 124.46) (diameter 0) (color 0 0 0 0)
-  )
   (junction (at 119.38 109.22) (diameter 0) (color 0 0 0 0)
   )
   (junction (at 148.59 80.01) (diameter 0) (color 0 0 0 0)
   )
-  (junction (at 109.22 82.55) (diameter 0) (color 0 0 0 0)
-  )
   (junction (at 148.59 121.92) (diameter 0) (color 0 0 0 0)
   )
@@
     (stroke (width 0) (type default))
   )
+  (wire (pts (xy 109.22 116.84) (xy 109.22 120.65))
+    (stroke (width 0) (type default))
+  )
   (wire (pts (xy 128.27 119.38) (xy 128.27 109.22))
     (stroke (width 0) (type default))
@@
     (stroke (width 0) (type default))
   )
-  (wire (pts (xy 109.22 82.55) (xy 129.54 82.55))
-    (stroke (width 0) (type default))
-  )
-  (wire (pts (xy 109.22 124.46) (xy 129.54 124.46))
+  (wire (pts (xy 113.03 124.46) (xy 129.54 124.46))
+    (stroke (width 0) (type default))
+  )
+  (wire (pts (xy 109.22 128.27) (xy 109.22 132.08))
     (stroke (width 0) (type default))
   )
@@
     (stroke (width 0) (type default))
   )
+  (wire (pts (xy 109.22 86.36) (xy 109.22 90.17))
+    (stroke (width 0) (type default))
+  )
+  (wire (pts (xy 113.03 82.55) (xy 129.54 82.55))
+    (stroke (width 0) (type default))
+  )
   (wire (pts (xy 128.27 77.47) (xy 128.27 67.31))
     (stroke (width 0) (type default))
@@
     (stroke (width 0) (type default))
   )
+  (wire (pts (xy 109.22 74.93) (xy 109.22 78.74))
+    (stroke (width 0) (type default))
+  )
   (wire (pts (xy 144.78 80.01) (xy 148.59 80.01))
     (stroke (width 0) (type default))
@@
     (stroke (width 0) (type default))
   )
-  (text "Dead Battery warning triggers at 2.79v/cell" (at 123.19 132.08 0)
+  (text "Dead Battery warning, adjustable" (at 123.19 132.08 0)
     (effects (font (size 1.27 1.27)) (justify left bottom))
   )
@@
     (effects (font (size 3 3)) (justify left bottom))
   )
-  (text "Low voltage warning triggers at 3.22v/cell" (at 121.92 91.44 0)
+  (text "Low Battery Warning, adjustable" (at 121.92 91.44 0)
     (effects (font (size 1.27 1.27)) (justify left bottom))
   )
@@
     )
   )
+  (symbol (lib_id "Device:R_Potentiometer") (at 109.22 82.55 0) (unit 1)
+    (in_bom yes) (on_board yes) (dnp no) (fields_autoplaced)
+    (property "Reference" "RV2" (at 106.68 81.28 0)
+      (effects (font (size 1.27 1.27)) (justify right))
+    )
+    (property "Value" "10k" (at 106.68 83.82 0)
+      (effects (font (size 1.27 1.27)) (justify right))
+    )
+    (property "Footprint" "" (at 109.22 82.55 0)
+      (effects (font (size 1.27 1.27)) hide)
+    )
+    (property "Datasheet" "~" (at 109.22 82.55 0)
+      (effects (font (size 1.27 1.27)) hide)
+    )
+    (pin "3")
+    (pin "2")
+    (pin "1")
+    (instances
+      (project "Baja_ECVT_controller"
+        (path "/c079eab7-726a-471f-be62-709191f368a5/bdd6113e-2452-49f0-9c6c-e5a49c773210"
+          (reference "RV2") (unit 1)
+        )
+      )
+    )
+  )
   (symbol (lib_id "power:+5V") (at 109.22 116.84 0) (unit 1)
     (in_bom yes) (on_board yes) (dnp no) (fields_autoplaced)
@@
       (effects (font (size 1.27 1.27)) (justify left))
     )
-    (property "Value" "2k2" (at 173.99 90.17 0)
+    (property "Value" "220" (at 173.99 90.17 0)
       (effects (font (size 1.27 1.27)) (justify left))
     )
@@
       (effects (font (size 1.27 1.27)) (justify left))
     )
-    (property "Value" "2k2" (at 173.99 132.08 0)
+    (property "Value" "220" (at 173.99 132.08 0)
       (effects (font (size 1.27 1.27)) (justify left))
     )
@@
       (effects (font (size 1.27 1.27)) (justify left))
     )
-    (property "Value" "8k2" (at 121.92 106.68 0)
+    (property "Value" "100k" (at 121.92 106.68 0)
       (effects (font (size 1.27 1.27)) (justify left))
     )
@@
     )
   )
-  (symbol (lib_id "Device:R") (at 109.22 128.27 0) (unit 1)
-    (in_bom yes) (on_board yes) (dnp no) (fields_autoplaced)
-    (property "Reference" "R14" (at 111.76 127 0)
-      (effects (font (size 1.27 1.27)) (justify left))
-    )
-    (property "Value" "6k8" (at 111.76 129.54 0)
-      (effects (font (size 1.27 1.27)) (justify left))
-    )
-    (property "Footprint" "" (at 107.442 128.27 90)
-      (effects (font (size 1.27 1.27)) hide)
-    )
-    (property "Datasheet" "~" (at 109.22 128.27 0)
-      (effects (font (size 1.27 1.27)) hide)
-    )
-    (pin "1")
-    (pin "2")
-    (instances
-      (project "Baja_ECVT_controller"
-        (path "/c079eab7-726a-471f-be62-709191f368a5"
-          (reference "R14") (unit 1)
-        )
-        (path "/c079eab7-726a-471f-be62-709191f368a5/bdd6113e-2452-49f0-9c6c-e5a49c773210"
-          (reference "R31") (unit 1)
-        )
-      )
-    )
-  )
-  (symbol (lib_id "Device:R") (at 109.22 78.74 0) (unit 1)
-    (in_bom yes) (on_board yes) (dnp no) (fields_autoplaced)
-    (property "Reference" "R9" (at 111.76 77.47 0)
-      (effects (font (size 1.27 1.27)) (justify left))
-    )
-    (property "Value" "2k2" (at 111.76 80.01 0)
-      (effects (font (size 1.27 1.27)) (justify left))
-    )
-    (property "Footprint" "" (at 107.442 78.74 90)
-      (effects (font (size 1.27 1.27)) hide)
-    )
-    (property "Datasheet" "~" (at 109.22 78.74 0)
-      (effects (font (size 1.27 1.27)) hide)
-    )
-    (pin "1")
-    (pin "2")
-    (instances
-      (project "Baja_ECVT_controller"
-        (path "/c079eab7-726a-471f-be62-709191f368a5"
-          (reference "R9") (unit 1)
-        )
-        (path "/c079eab7-726a-471f-be62-709191f368a5/bdd6113e-2452-49f0-9c6c-e5a49c773210"
-          (reference "R28") (unit 1)
-        )
-      )
-    )
-  )
   (symbol (lib_id "Device:R") (at 148.59 118.11 0) (unit 1)
     (in_bom yes) (on_board yes) (dnp no) (fields_autoplaced)
@@
     )
   )
-  (symbol (lib_id "Device:R") (at 109.22 120.65 0) (unit 1)
-    (in_bom yes) (on_board yes) (dnp no) (fields_autoplaced)
-    (property "Reference" "R13" (at 111.76 119.38 0)
-      (effects (font (size 1.27 1.27)) (justify left))
-    )
-    (property "Value" "4k7" (at 111.76 121.92 0)
-      (effects (font (size 1.27 1.27)) (justify left))
-    )
-    (property "Footprint" "" (at 107.442 120.65 90)
-      (effects (font (size 1.27 1.27)) hide)
-    )
-    (property "Datasheet" "~" (at 109.22 120.65 0)
-      (effects (font (size 1.27 1.27)) hide)
-    )
-    (pin "1")
-    (pin "2")
-    (instances
-      (project "Baja_ECVT_controller"
-        (path "/c079eab7-726a-471f-be62-709191f368a5"
-          (reference "R13") (unit 1)
-        )
-        (path "/c079eab7-726a-471f-be62-709191f368a5/bdd6113e-2452-49f0-9c6c-e5a49c773210"
-          (reference "R30") (unit 1)
-        )
-      )
-    )
-  )
   (symbol (lib_id "Device:R") (at 119.38 63.5 0) (unit 1)
     (in_bom yes) (on_board yes) (dnp no) (fields_autoplaced)
@@
       (effects (font (size 1.27 1.27)) (justify left))
     )
-    (property "Value" "8k2" (at 121.92 64.77 0)
+    (property "Value" "100k" (at 121.92 64.77 0)
       (effects (font (size 1.27 1.27)) (justify left))
     )
@@
       (effects (font (size 1.27 1.27)) (justify left))
     )
-    (property "Value" "2k2" (at 121.92 114.3 0)
+    (property "Value" "10k" (at 121.92 114.3 0)
       (effects (font (size 1.27 1.27)) (justify left))
     )
@@
     )
   )
-  (symbol (lib_id "Device:R") (at 109.22 86.36 0) (unit 1)
-    (in_bom yes) (on_board yes) (dnp no) (fields_autoplaced)
-    (property "Reference" "R10" (at 111.76 85.09 0)
-      (effects (font (size 1.27 1.27)) (justify left))
-    )
-    (property "Value" "4k7" (at 111.76 87.63 0)
-      (effects (font (size 1.27 1.27)) (justify left))
-    )
-    (property "Footprint" "" (at 107.442 86.36 90)
-      (effects (font (size 1.27 1.27)) hide)
-    )
-    (property "Datasheet" "~" (at 109.22 86.36 0)
-      (effects (font (size 1.27 1.27)) hide)
-    )
-    (pin "1")
-    (pin "2")
-    (instances
-      (project "Baja_ECVT_controller"
-        (path "/c079eab7-726a-471f-be62-709191f368a5"
-          (reference "R10") (unit 1)
-        )
-        (path "/c079eab7-726a-471f-be62-709191f368a5/bdd6113e-2452-49f0-9c6c-e5a49c773210"
-          (reference "R29") (unit 1)
-        )
-      )
-    )
-  )
   (symbol (lib_id "Device:R") (at 160.02 121.92 90) (unit 1)
     (in_bom yes) (on_board yes) (dnp no) (fields_autoplaced)
@@
       (effects (font (size 1.27 1.27)) (justify left))
     )
-    (property "Value" "2k2" (at 121.92 72.39 0)
+    (property "Value" "10k" (at 121.92 72.39 0)
       (effects (font (size 1.27 1.27)) (justify left))
     )
@@
         )
       )
+    )
+  )
+  (symbol (lib_id "Device:R_Potentiometer") (at 109.22 124.46 0) (unit 1)
+    (in_bom yes) (on_board yes) (dnp no) (fields_autoplaced)
+    (property "Reference" "RV1" (at 106.68 123.19 0)
+      (effects (font (size 1.27 1.27)) (justify right))
+    )
+    (property "Value" "10k" (at 106.68 125.73 0)
+      (effects (font (size 1.27 1.27)) (justify right))
+    )
+    (property "Footprint" "" (at 109.22 124.46 0)
+      (effects (font (size 1.27 1.27)) hide)
+    )
+    (property "Datasheet" "~" (at 109.22 124.46 0)
+      (effects (font (size 1.27 1.27)) hide)
+    )
+    (pin "3")
+    (pin "2")
+    (pin "1")
+    (instances
+      (project "Baja_ECVT_controller"
+        (path "/c079eab7-726a-471f-be62-709191f368a5/bdd6113e-2452-49f0-9c6c-e5a49c773210"
+          (reference "RV1") (unit 1)
+        )
+      )

Commit message: Add files via upload
Parts:
- added C11: 100n, Capacitor_SMD:C_0402_1005Metric, symbol Device:C
- Q1, Q2: footprint (none) -> Package_TO_SOT_SMD:SOT-323_SC-70
- R11, R12, R15, R16, R17, R18, R5, R6, R7, R8: footprint (none) -> Resistor_SMD:R_0402_1005Metric
- RV1, RV2: footprint (none) -> Potentiometer_THT:Potentiometer_Bourns_3386F_Vertical
- U3: footprint (none) -> Package_SO:SOIC-8_3.9x4.9mm_P1.27mm
Connections:
- net +5V: now also C11.1
- net GND: now also C11.2
- net +BATT renamed Vdrive
