File: conn.kicad_sch (KiCad schematic)
At the start: 5 parts, among them J2 Conn_01x02_Pin, J5 Conn_01x02_Pin, J7 Conn_01x24_Pin

Commit message: Add files via upload
Connections:
- net Encoder1_2 is gone; now on net GND: J7.3 (Pin_3)
- net GND: no longer J7.4 (Pin_4)
- net Encoder1_1 renamed Hall_Effect
- no-connect marks 1 -> 2
Other:
- moved on the sheet: JP1, R5
Changed lines of the file:
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@@
 (kicad_sch (version 20230121) (generator eeschema)
   (paper "A5" portrait)
-  (junction (at 121.92 144.78) (diameter 0) (color 0 0 0 0)
-  )
-  (junction (at 121.92 127) (diameter 0) (color 0 0 0 0)
+  (junction (at 115.57 144.78) (diameter 0) (color 0 0 0 0)
+  )
+  (junction (at 115.57 127) (diameter 0) (color 0 0 0 0)
   )
   (no_connect (at 71.12 107.95))
-  (wire (pts (xy 118.11 133.35) (xy 118.11 127))
+  (no_connect (at 71.12 85.09))
+  (wire (pts (xy 111.76 133.35) (xy 111.76 127))
     (stroke (width 0) (type default))
   )
@@
     (stroke (width 0) (type default))
   )
-  (wire (pts (xy 85.09 82.55) (xy 71.12 82.55))
-    (stroke (width 0) (type default))
-  )
-  (wire (pts (xy 91.44 74.93) (xy 85.09 74.93))
-    (stroke (width 0) (type default))
-  )
   (wire (pts (xy 71.12 105.41) (xy 113.03 105.41))
     (stroke (width 0) (type default))
@@
     (stroke (width 0) (type default))
   )
-  (wire (pts (xy 118.11 144.78) (xy 118.11 135.89))
+  (wire (pts (xy 111.76 144.78) (xy 111.76 135.89))
     (stroke (width 0) (type default))
   )
@@
     (stroke (width 0) (type default))
   )
-  (wire (pts (xy 118.11 127) (xy 121.92 127))
+  (wire (pts (xy 111.76 127) (xy 115.57 127))
+    (stroke (width 0) (type default))
+  )
+  (wire (pts (xy 71.12 82.55) (xy 85.09 82.55))
     (stroke (width 0) (type default))
   )
@@
     (stroke (width 0) (type default))
   )
-  (wire (pts (xy 87.63 85.09) (xy 87.63 77.47))
+  (wire (pts (xy 85.09 82.55) (xy 85.09 74.93))
     (stroke (width 0) (type default))
   )
@@
     (stroke (width 0) (type default))
   )
-  (wire (pts (xy 121.92 144.78) (xy 123.19 144.78))
+  (wire (pts (xy 115.57 144.78) (xy 116.84 144.78))
     (stroke (width 0) (type default))
   )
@@
     (stroke (width 0) (type default))
   )
-  (wire (pts (xy 121.92 127) (xy 123.19 127))
+  (wire (pts (xy 115.57 127) (xy 116.84 127))
     (stroke (width 0) (type default))
   )
@@
     (stroke (width 0) (type default))
   )
-  (wire (pts (xy 118.11 144.78) (xy 121.92 144.78))
+  (wire (pts (xy 111.76 144.78) (xy 115.57 144.78))
     (stroke (width 0) (type default))
   )
@@
     (stroke (width 0) (type default))
   )
-  (wire (pts (xy 87.63 85.09) (xy 71.12 85.09))
-    (stroke (width 0) (type default))
-  )
   (wire (pts (xy 80.01 68.58) (xy 80.01 77.47))
     (stroke (width 0) (type default))
@@
     (stroke (width 0) (type default))
   )
-  (wire (pts (xy 118.11 135.89) (xy 71.12 135.89))
+  (wire (pts (xy 111.76 135.89) (xy 71.12 135.89))
     (stroke (width 0) (type default))
   )
@@
     (stroke (width 0) (type default))
   )
-  (wire (pts (xy 85.09 74.93) (xy 85.09 82.55))
-    (stroke (width 0) (type default))
-  )
-  (wire (pts (xy 71.12 133.35) (xy 118.11 133.35))
+  (wire (pts (xy 71.12 133.35) (xy 111.76 133.35))
+    (stroke (width 0) (type default))
+  )
+  (wire (pts (xy 104.14 74.93) (xy 104.14 76.2))
     (stroke (width 0) (type default))
   )
@@
     (stroke (width 0) (type default))
   )
-  (wire (pts (xy 87.63 77.47) (xy 104.14 77.47))
+  (wire (pts (xy 85.09 74.93) (xy 104.14 74.93))
     (stroke (width 0) (type default))
   )
@@
     )
   )
-  (global_label "Encoder1_1" (shape input) (at 91.44 71.12 0) (fields_autoplaced)
-    (effects (font (size 1.27 1.27)) (justify left))
-    (property "Intersheetrefs" "${INTERSHEET_REFS}" (at 105.3712 71.12 0)
-      (effects (font (size 1.27 1.27)) (justify left) hide)
-    )
-  )
   (global_label "Dead_Batt_ind" (shape input) (at 71.12 130.81 0) (fields_autoplaced)
     (effects (font (size 1.27 1.27)) (justify left))
@@
     )
   )
-  (global_label "Encoder1_2" (shape input) (at 91.44 74.93 0) (fields_autoplaced)
-    (effects (font (size 1.27 1.27)) (justify left))
-    (property "Intersheetrefs" "${INTERSHEET_REFS}" (at 105.3712 74.93 0)
-      (effects (font (size 1.27 1.27)) (justify left) hide)
-    )
-  )
-  (global_label "CAN_-" (shape input) (at 123.19 144.78 0) (fields_autoplaced)
-    (effects (font (size 1.27 1.27)) (justify left))
-    (property "Intersheetrefs" "${INTERSHEET_REFS}" (at 132.4043 144.78 0)
+  (global_label "CAN_-" (shape input) (at 116.84 144.78 0) (fields_autoplaced)
+    (effects (font (size 1.27 1.27)) (justify left))
+    (property "Intersheetrefs" "${INTERSHEET_REFS}" (at 126.0543 144.78 0)
       (effects (font (size 1.27 1.27)) (justify left) hide)
     )
@@
     )
   )
-  (global_label "CAN_+" (shape input) (at 123.19 127 0) (fields_autoplaced)
-    (effects (font (size 1.27 1.27)) (justify left))
-    (property "Intersheetrefs" "${INTERSHEET_REFS}" (at 132.4043 127 0)
+  (global_label "CAN_+" (shape input) (at 116.84 127 0) (fields_autoplaced)
+    (effects (font (size 1.27 1.27)) (justify left))
+    (property "Intersheetrefs" "${INTERSHEET_REFS}" (at 126.0543 127 0)
       (effects (font (size 1.27 1.27)) (justify left) hide)
     )
@@
     )
   )
+  (global_label "Hall_Effect" (shape input) (at 91.44 71.12 0) (fields_autoplaced)
+    (effects (font (size 1.27 1.27)) (justify left))
+    (property "Intersheetrefs" "${INTERSHEET_REFS}" (at 104.706 71.12 0)
+      (effects (font (size 1.27 1.27)) (justify left) hide)
+    )
+  )
   (global_label "GPIO_2" (shape input) (at 71.12 120.65 0) (fields_autoplaced)
     (effects (font (size 1.27 1.27)) (justify left))
@@
     )
   )
-  (symbol (lib_id "power:GND") (at 104.14 77.47 0) (mirror y) (unit 1)
-    (in_bom yes) (on_board yes) (dnp no) (fields_autoplaced)
-    (property "Reference" "#PWR061" (at 104.14 83.82 0)
-      (effects (font (size 1.27 1.27)) hide)
-    )
-    (property "Value" "GND" (at 104.14 82.55 0)
-      (effects (font (size 1.27 1.27)))
-    )
-    (property "Footprint" "" (at 104.14 77.47 0)
-      (effects (font (size 1.27 1.27)) hide)
-    )
-    (property "Datasheet" "" (at 104.14 77.47 0)
+  (symbol (lib_id "power:GND") (at 104.14 76.2 0) (mirror y) (unit 1)
+    (in_bom yes) (on_board yes) (dnp no) (fields_autoplaced)
+    (property "Reference" "#PWR061" (at 104.14 82.55 0)
+      (effects (font (size 1.27 1.27)) hide)
+    )
+    (property "Value" "GND" (at 104.14 81.28 0)
+      (effects (font (size 1.27 1.27)))
+    )
+    (property "Footprint" "" (at 104.14 76.2 0)
+      (effects (font (size 1.27 1.27)) hide)
+    )
+    (property "Datasheet" "" (at 104.14 76.2 0)
       (effects (font (size 1.27 1.27)) hide)
     )
@@
     )
   )
-  (symbol (lib_id "Device:R") (at 121.92 130.81 0) (unit 1)
-    (in_bom yes) (on_board yes) (dnp no) (fields_autoplaced)
-    (property "Reference" "R5" (at 124.46 129.54 0)
+  (symbol (lib_id "Device:R") (at 115.57 130.81 0) (unit 1)
+    (in_bom yes) (on_board yes) (dnp no) (fields_autoplaced)
+    (property "Reference" "R5" (at 118.11 129.54 0)
       (effects (font (size 1.27 1.27)) (justify left))
     )
-    (property "Value" "120" (at 124.46 132.08 0)
+    (property "Value" "120" (at 118.11 132.08 0)
       (effects (font (size 1.27 1.27)) (justify left))
     )
-    (property "Footprint" "" (at 120.142 130.81 90)
-      (effects (font (size 1.27 1.27)) hide)
-    )
-    (property "Datasheet" "~" (at 121.92 130.81 0)
+    (property "Footprint" "" (at 113.792 130.81 90)
+      (effects (font (size 1.27 1.27)) hide)
+    )
+    (property "Datasheet" "~" (at 115.57 130.81 0)
       (effects (font (size 1.27 1.27)) hide)
     )
@@
     )
   )
-  (symbol (lib_id "Jumper:Jumper_2_Bridged") (at 121.92 139.7 90) (unit 1)
-    (in_bom yes) (on_board yes) (dnp no) (fields_autoplaced)
-    (property "Reference" "JP1" (at 123.19 138.43 90)
+  (symbol (lib_id "Jumper:Jumper_2_Bridged") (at 115.57 139.7 90) (unit 1)
+    (in_bom yes) (on_board yes) (dnp no) (fields_autoplaced)
+    (property "Reference" "JP1" (at 116.84 138.43 90)
       (effects (font (size 1.27 1.27)) (justify right))
     )
-    (property "Value" "Jumper_2_Bridged" (at 123.19 140.97 90)
+    (property "Value" "Jumper_2_Bridged" (at 116.84 140.97 90)
       (effects (font (size 1.27 1.27)) (justify right))
     )
-    (property "Footprint" "" (at 121.92 139.7 0)
-      (effects (font (size 1.27 1.27)) hide)
-    )
-    (property "Datasheet" "~" (at 121.92 139.7 0)
-      (effects (font (size 1.27 1.27)) hide)
-    )
+    (property "Footprint" "" (at 115.57 139.7 0)
+      (effects (font (size 1.27 1.27)) hide)
+    )
+    (property "Datasheet" "~" (at 115.57 139.7 0)
+      (effects (font (size 1.27 1.27)) hide)
+    )

Commit message: Add files via upload
Parts:
- removed JP1: Jumper_2_Bridged, symbol Jumper:Jumper_2_Bridged
- J2, J5: footprint (none) -> Connector_Molex:Molex_Mega-Fit_76829-0002_2x01_P5.70mm_Vertical
- J7: footprint (none) -> Connector_Molex:Molex_Micro-Fit_3.0_43045-2412_2x12_P3.00mm_Vertical
- R5: footprint (none) -> Resistor_SMD:R_0603_1608Metric
Connections:
- net +5V: now also J7.21 (Pin_21); no longer J7.9 (Pin_9)
- net CAN_+: now also J7.12 (Pin_12), R5.2; no longer J7.23 (Pin_23), R5.1
- net CAN_-: now also J7.11 (Pin_11), R5.1; no longer J7.24 (Pin_24)
- net Dead_Batt_ind: now also J7.10 (Pin_10); no longer J7.22 (Pin_22)
- net Encoder2_1: now also J7.22 (Pin_22); no longer J7.10 (Pin_10), J7.6 (Pin_6)
- net Encoder2_2: now also J7.23 (Pin_23); no longer J7.11 (Pin_11), J7.7 (Pin_7)
- net GND: now also J7.24 (Pin_24); no longer J7.12 (Pin_12)
- net Low_Batt_ind: now also J7.9 (Pin_9); no longer J7.21 (Pin_21)
- new net Encoder1_1: J7.6 (Pin_6)
- new net Encoder1_2: J7.7 (Pin_7)
Other:
- moved on the sheet: R5
