File: motor_control.kicad_sch (KiCad schematic)
At the start: 29 parts, among them Q3 PMOS, Q4 PMOS, Q5 NMOS, Q6 NMOS, U4 INA2180A2IDGKR, U5 IR2103STRPBF, U6 IR2103STRPBF

Commit message: Add files via upload
Connections:
- net +BATT: now also C34.1, C36.1, CR1.1, CR2.1, U5.8 (VB), U6.8 (VB); no longer C33.1, C35.1, CR1.2, CR2.2, U5.1 (VCC), U6.1 (VCC)
- new net +12V: C33.1, C35.1, CR1.2, CR2.2, U5.1 (VCC), U6.1 (VCC)

Commit message: Add files via upload
Parts:
- removed C31: 1n, symbol Device:C
- removed CR3, CR4, CR5, CR6: DSS110U, CR_SOD-123FL_SME, symbol My_diodes:DSS110U
- removed Q3, Q4: PMOS, symbol Simulation_SPICE:PMOS
- removed R20: 1m, symbol Device:R
- removed R21: 1k, symbol Device:R
- removed U4: INA2180A2IDGKR, DGK8_TEX, symbol curr_sense_amp:INA2180A2IDGKR
- added Q5 (x2): NMOS, Package_TO_SOT_SMD:TO-252-2, symbol Simulation_SPICE:NMOS
- added U10: INA180A2IDBVR, single_curr_sense:DBV0005A_N, symbol single_curr_sense:INA180A2IDBVR
- C30, C32: footprint (none) -> Capacitor_SMD:C_0402_1005Metric
- C33, C34, C35, C36: footprint (none) -> Capacitor_SMD:C_0603_1608Metric
- C37: footprint (none) -> Capacitor_THT:CP_Radial_D6.3mm_P2.50mm
- CR1, CR2: footprint CR_SOD-123FL_SME -> Diode_SMD:D_SOD-123F
- Q5, Q6: footprint (none) -> Package_TO_SOT_SMD:TO-252-2
- R19: footprint (none) -> Resistor_SMD:R_2512_6332Metric
- R22: footprint (none) -> Resistor_SMD:R_0402_1005Metric
- R23, R24, R25, R26: footprint (none) -> Resistor_SMD:R_0805_2012Metric
- U5, U6: footprint IR2103STRPBF:SOIC127P600X175-8N -> H_Bridge:SOIC127P600X175-8N
Connections:
- net GND: now also U10.4 (IN-)
- net GNDA: now also U10.2 (GND); no longer Q6.3 (S)
- net Motor_A: now also Q5.2 (D), Q5.3 (S); no longer Q5.1 (D)
- net Motor_B: now also Q6.2 (D), Q5.3 (S); no longer Q6.1 (D)
- net VDDA: now also U10.5 (VS)
- net at Q5.3 (S), R19.1: now also Q6.3 (S), U10.3 (IN+)
- net at R22.2: now also U10.1 (OUT)
- net at R23.2: now also Q5.1 (G)
- net at R24.2: now also Q5.1 (G); no longer Q5.2 (G)
- net at R26.1: now also Q6.1 (G); no longer Q6.2 (G)
- net at R25.1: now also Q5.1 (G)
- net +BATT renamed Vdrive
- net Vdrive: now also Q5.2 (D), Q5.2 (D)
Other:
- note added: "Fix current sense"
- moved on the sheet: C30, C32, R19, R22
