File: power_sup.kicad_sch (KiCad schematic)
At the start: 10 parts, among them U2 AZ1117-3.3

Commit message: Add files via upload
Parts:
- removed U2: AZ1117-3.3, symbol Regulator_Linear:AZ1117-3.3
- added C28, C29: 1u, symbol Device:C
- added D1: LED, symbol Device:LED
- added D2: D_Schottky_KAA, symbol Device:D_Schottky_KAA
- added F1: 15A, symbol Device:Fuse
- added R6: 1k, symbol Device:R
- added U2, U3: AP7370-50FDC, Package_DFN_QFN:DFN-6-1EP_2x2mm_P0.65mm_EP1.01x1.7mm, symbol Regulator_Linear:AP7370-50FDC
- C28: value 22u -> 1u
- C29: value 10u -> 1u
- PS1: value K7805-500R3 -> LMP78_12-1.0R; footprint K7803-500R3:CONV_K7803-500R3 -> (none); MANUFACTURER Mornsun -> (none); MAXIMUM_PACKAGE_HEIGHT 10.41 mm -> (none); PARTREV 2020.12.17-A/7 -> (none); STANDARD Manufacturer Recommendations -> (none)
Connections:
- net +3.3V: now also C28.1, U2.1 (VO); no longer C28.1
- net +5V: now also C28.1, C29.1, R6.1, U2.6 (VI), U3.1 (VO); no longer C24.1, C29.1, PS1.3 (+VO)
- net +BATT: now also F1.1; no longer C9.1, PS1.1 (VIN)
- net GND: now also C28.2, C29.2, D1.1 (K), U2.3 (GND), U2.7 (GND), U3.3 (GND), U3.7 (GND)
- new net: D2.2 (A), D2.3 (A), F1.2
- new net: D1.2 (A), R6.2
- new net: C9.1, D2.1 (K), PS1.1 (VIN)
- new net +12V: C24.1, C29.1, PS1.3 (+VO), U3.6 (VI)
Other:
- note added: "Green LED for power indication"
- moved on the sheet: C24, C25, C26, C27, C28, C29, C9, FB1, PS1

Commit message: Add files via upload
Parts:
- removed F1: 15A, symbol Device:Fuse
- added F2: 3557-2, fuse_block:FUSE_3557-2, symbol fuse:3557-2
- added NT1: NetTie_2, NetTie:NetTie-2_SMD_Pad2.0mm, symbol Device:NetTie_2
- C24, C9: footprint (none) -> Capacitor_SMD:C_1206_3216Metric
- C25, C26, C28, C29: footprint (none) -> Capacitor_SMD:C_0603_1608Metric
- C27: footprint (none) -> Capacitor_SMD:C_0402_1005Metric
- D1: footprint (none) -> LED_SMD:LED_0603_1608Metric
- D2: footprint (none) -> shottky:TO-277B_MBR1560S_SME
- FB1, R6: footprint (none) -> Resistor_SMD:R_0402_1005Metric
- PS1: footprint (none) -> SMPS:CONV_K7803-500R3
- U2: value AP7370-50FDC -> AP7370-33FDC
Connections:
- net +BATT: now also F2.1_1
- net GND: now also NT1.2; no longer C26.2, C27.2
- net Vdrive: now reaches D2.2 (A), D2.3 (A)
- net Vdrive: now also F2.2_1
- new net GNDA: C26.2, C27.2, NT1.1
